Commit message: added table mount

File: ridgeback_franka_description/urdf/ridgeback_panda_hand_description.urdf.xacro (robot description, xacro)
@@ -8,8 +8,65 @@
   <xacro:include filename="$(find franka_description)/robots/gzplugin_grasp_fix.xacro"/>
   <xacro:include filename="$(find franka_description)/robots/panda.transmission.xacro"/>
+  <link name="table_top_link">
+    <visual>
+      <geometry>
+        <mesh filename="package://ridgeback_franka_description/meshes/hams-table-top.stl" />
+      </geometry>
+      <material name="black" />
+    </visual>
+    <collision>
+      <origin xyz="0 0 0" rpy="0 0 0"/>
+      <geometry>
+        <mesh filename="package://ridgeback_franka_description/meshes/hams-table-top.stl" />
+      </geometry>
+    </collision>
+  </link>
+  <link name="table_legs_link">
+    <visual>
+      <geometry>
+        <mesh filename="package://ridgeback_franka_description/meshes/hams-table-legs.stl" />
+      </geometry>
+      <material name="light_grey" />
+    </visual>
+    <collision>
+      <origin xyz="0 0 0" rpy="0 0 0"/>
+      <geometry>
+        <mesh filename="package://ridgeback_franka_description/meshes/hams-table-legs.stl" />
+      </geometry>
+    </collision>
+  </link>
+  <joint name="table_top_joint" type="fixed">
+    <parent link="mid_mount" />
+    <child link="table_top_link" />
+    <origin xyz="0 0 0.60635" rpy="0 0 0"/>
+  </joint>
+  <joint name="table_legs_joint" type="fixed">
+    <parent link="mid_mount" />
+    <child link="table_legs_link" />
+    <origin xyz="0 0 0.60635" rpy="0 0 0"/>
+  </joint>
+  <link name="arm_mount_link">
+    <visual>
+      <geometry>
+        <mesh filename="package://ridgeback_franka_description/meshes/hams-arm-mount.stl" />
+      </geometry>
+      <material name="black" />
+    </visual>
+    <collision>
+      <origin xyz="0 0 0" rpy="0 0 0"/>
+      <geometry>
+        <mesh filename="package://ridgeback_franka_description/meshes/hams-arm-mount.stl" />
+      </geometry>
+    </collision>
+  </link>
   <joint name="arm_mount_joint" type="fixed">
     <parent link="mid_mount" />
+    <child link="arm_mount_link" />
+    <origin xyz="-.27913 0 $(optenv RIDGEBACK_ARM_HEIGHT 0.31)" rpy="0 0 $(optenv RIDGEBACK_ARM_ANGLE 0.0)"/>
+  </joint>
+  <joint name="arm_mount_joint_2" type="fixed">
+    <parent link="arm_mount_link" />
     <child link="franka_mount_link" />
-    <origin xyz="$(optenv RIDGEBACK_FRANKA_XYZ 0.21 0.0 0.0)" rpy="$(optenv RIDGEBACK_FRANKA_RPY 0 0 0)"/>
+    <origin xyz="$(optenv RIDGEBACK_FRANKA_XYZ 0.0 0.0 0.0)" rpy="$(optenv RIDGEBACK_FRANKA_RPY 0 0 0)"/>
   </joint>
   <link name="franka_mount_link" />
